Commit message: lidar works and odom frame appears in rviz2

File: urdf/two_wheeled_robot.urdf (robot description, URDF)
Before this commit: robot two_wheeled_robot, 6 links, 5 joints
Links:
- link camera_link: geometry visual cylinder length=.02 radius=.02

Commit message: working better

File: urdf/two_wheeled_robot.urdf (robot description, URDF)
Before this commit: robot two_wheeled_robot, 6 links, 5 joints
Links:
- link imu_link: geometry visual box size=0.01 0.01 0.001
Joints:
- joint imu_joint: origin xyz=-0.10 0 0.05 rpy=0 0 0 -> xyz=-0.08 -0.06 0.05 rpy=0 0 0

Commit message: ekf node working better

File: urdf/two_wheeled_robot.urdf (robot description, URDF)
Before this commit: robot two_wheeled_robot, 6 links, 5 joints
Links:
- removed link front_caster
- added link back_plate_link; collision box size=${.02} ${base_width} ${.002}; visual box size=${.02} ${base_width} ${.002}
- added link rear_caster; collision sphere radius=${caster_radius}; visual sphere radius=0.05
Joints:
- added joint back_plate_joint: type fixed, parent base_link, child back_plate_link, origin xyz=${(base_length/-2.)-.01} 0.0 0.10 rpy=0 0 0
- joint caster_joint: child front_caster -> rear_caster
